File: Beacon_and_eggs/_restore_backup_2026-05-14T11-46-56-307/Beacon_and_eggs.kicad_pcb (KiCad board)
At the start: 4 copper layers, 40 x 80 mm, 73 parts, among them J1 USB_C_Receptacle_USB2.0_16P, J2 Conn_01x03_Pin, J3 Conn_01x02_Pin, Q1 NTA4151P, Q2 NTA4153N, U1 SA868S, U2 STM32F411CEU6TR, U3 ADXL343, U4 MIC5528-3.3YMX-TR, U6 BQ24070RHLR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

Commit message: fixed accel. pinouts, added 10k resistor to TS of U6
Parts:
- removed REF** (x2): MountingHole_2.2mm_M2_ISO14580_Pad_TopBottom, MountingHole:MountingHole_2.2mm_M2_ISO14580_Pad_TopBottom
